Commit message: simulation ready

File: legRBDL.urdf (robot description, URDF)
Before this commit: robot leg, 7 links, 6 joints
Links:
- removed link foot
Joints:
- removed joint foot_fixed

Commit message: Code clean up

File: legRBDL.urdf (robot description, URDF)
Before this commit: robot leg, 6 links, 5 joints
Links:
- link jump: mass 0.002 -> 2

Commit message: plots added

File: legRBDL.urdf (robot description, URDF)
Before this commit: robot leg, 6 links, 5 joints
Links:
- link trunk_inertia: mass None -> 100

Commit message: PD controller on slip

File: legRBDL.urdf (robot description, URDF)
Before this commit: robot leg, 6 links, 5 joints
Joints:
- joint jumper: origin xyz=0 0 0.9 rpy=0 0 0 -> xyz=0 0 0.6 rpy=0 0 0

Commit message: PD controller for stance mode added

File: legRBDL.urdf (robot description, URDF)
Before this commit: robot leg, 6 links, 5 joints
Links:
- link jump: mass 2 -> 2.18

Commit message: extract data added for H=0.46

File: legRBDL.urdf (robot description, URDF)
Before this commit: robot leg, 6 links, 5 joints
Joints:
- joint jumper: origin xyz=0 0 0.6 rpy=0 0 0 -> xyz=0 0 0.46 rpy=0 0 0
