Commit message: simulation data to hardware

File: data_0.4/legRBDL.urdf (robot description, URDF)
Before this commit: robot leg, 6 links, 5 joints
Joints:
- joint jumper: origin xyz=0 0 0.40 rpy=0 0 0 -> xyz=0 0 0.4 rpy=0 0 0

File: data_0.4/leg_RBDL.urdf (robot description, URDF)
Before this commit: robot leg, 6 links, 5 joints
Links:
- removed link jump
- removed link trunk_inertia
- added link foot, mass 0.005; collision sphere radius=0.025; visual sphere radius=0.025
- added link world, mass 100
- link trunk: geometry collision box size=0.075 0.06 0.09; visual box size=0.075 0.06 0.09
Joints:
- removed joint jumper
- removed joint trunk_to_trunk_inertia
- added joint foot_fixed: type fixed, parent calf, child foot, origin xyz=0 0 -0.240 rpy=0 0 0, axis 0 1 0, limit lower=-3.14159265359 upper=3.14159265359 effort=20 velocity=10.6
- added joint trunk_to_world: type fixed, parent world, child trunk, origin xyz=0 0 0 rpy=0 0 0
- joint hip_joint: limit lower=-0.872664625997 upper=1.0471975512 effort=20 velocity=1.6 -> lower=-3.14 upper=3.14 effort=20 velocity=1.6; origin xyz=0.05 0 0 rpy=0 0 0 -> xyz=0.025 0 0 rpy=0 0 0; parent jump -> trunk
